Commit message: update example

File: model/dual_arm_model/dual_arm_model.urdf (robot description, URDF)
Before this commit: robot dual_arm_model_new, 24 links, 23 joints
Links:
- link base_link: geometry collision mesh filename=package://dual_arm_model/meshes/base_link_collisions.obj scale=1. 1. 1.; visual mesh filename=package://dual_arm_model/meshes/base_link_visuals.obj scale=1. 1. 1.
- link base_link_inertia1: geometry collision mesh filename=package://dual_arm_model/meshes/collision/base.stl scale=1. 1. 1.; visual mesh filename=package://dual_arm_model/meshes/visual/base.dae scale=1. 1. 1.
- link forearm_link: geometry collision mesh filename=package://dual_arm_model/meshes/forearm_link_collisions.obj scale=1. 1. 1.; visual mesh filename=package://dual_arm_model/meshes/forearm_link_visuals.obj scale=1. 1. 1.
- link forearm_link1: geometry collision mesh filename=package://dual_arm_model/meshes/collision/forearm.stl scale=1. 1. 1.; visual mesh filename=package://dual_arm_model/meshes/visual/forearm.dae scale=1. 1. 1.
- link shoulder_link: geometry collision mesh filename=package://dual_arm_model/meshes/shoulder_link_collisions.obj scale=1. 1. 1.; visual mesh filename=package://dual_arm_model/meshes/shoulder_link_visuals.obj scale=1. 1. 1.
- link shoulder_link1: geometry collision mesh filename=package://dual_arm_model/meshes/collision/shoulder.stl scale=1. 1. 1.; visual mesh filename=package://dual_arm_model/meshes/visual/shoulder.dae scale=1. 1. 1.
- link upper_arm_link: geometry collision mesh filename=package://dual_arm_model/meshes/upper_arm_link_collisions.o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 scale=1. 1. 1.; visual mesh filename=package://dual_arm_model/meshes/upper_arm_link_visuals.obj scale=1. 1. 1.
- link upper_arm_link1: geometry collision mesh filename=package://dual_arm_model/meshes/collision/upperarm.stl scale=1. 1. 1.; visual mesh filename=package://dual_arm_model/meshes/visual/upperarm.dae scale=1. 1. 1.
- link wrist_1_link: geometry collision mesh filename=package://dual_arm_model/meshes/wrist_1_link_collisions.obj scale=1. 1. 1.; visual mesh filename=package://dual_arm_model/meshes/wrist_1_link_visuals.obj scale=1. 1. 1.
- link wrist_1_link1: geometry collision mesh filename=package://dual_arm_model/meshes/collision/wrist1.stl scale=1. 1. 1.; visual mesh filename=package://dual_arm_model/meshes/visual/wrist1.dae scale=1. 1. 1.
- link wrist_2_link: geometry collision mesh filename=package://dual_arm_model/meshes/wrist_2_link_collisions.obj scale=1. 1. 1.; visual mesh filename=package://dual_arm_model/meshes/wrist_2_link_visuals.obj scale=1. 1. 1.
- link wrist_2_link1: geometry collision mesh filename=package://dual_arm_model/meshes/collision/wrist2.stl scale=1. 1. 1.; visual mesh filename=package://dual_arm_model/meshes/visual/wrist2.dae scale=1. 1. 1.
- link wrist_3_link1: geometry collision mesh filename=package://dual_arm_model/meshes/collision/wrist3.stl scale=1. 1. 1.; visual mesh filename=package://dual_arm_model/meshes/visual/wrist3.dae scale=1. 1. 1.

File: model/plane/big_plane1.urdf (robot description, URDF)
Before this commit: robot plane, 1 links, 0 joints
Links:
- link baseLink: geometry visual mesh filename=cube.obj scale=0.5 1.5 0.012

File: model/plane/big_plane2.urdf (robot description, URDF)
Before this commit: robot plane, 1 links, 0 joints
Links:
- link baseLink: geometry visual mesh filename=cube.obj scale=0.5 0.012 0.5

File: model/plane/thine_plane.urdf (robot description, URDF)
Before this commit: robot plane, 1 links, 0 joints
Links:
- link baseLink: geometry visual mesh filename=cube.obj scale=0.24 0.21 0.012
