Commit message: update some example

File: model/dual_panda_model/dual_panda_r9_urdf.urdf (robot description, URDF)
Before this commit: robot dual_panda_urdf, 27 links, 26 joints
Joints:
- joint left_panda_root_joint: origin xyz=-0.035 0.75 0.07 rpy=0. 0. -1.5707964 -> xyz=0.035 0.75 0.07 rpy=0. 0. -1.5707964
- joint right_panda_root_joint: origin xyz=-0.035 -0.75 0.07 rpy=0. 0. 1.5707963 -> xyz=0.035 -0.75 0.07 rpy=0. 0. 1.5707963
